Commit message: split xacros into multiple files

File: src/my_robot_description/urdf/my_robot.urdf.xacro (robot description, xacro)
@@ -1,70 +1,5 @@
 <?xml version="1.0"?>
 <robot name="my_robot" xmlns:xacro="http://www.ros.org/wiki/xacro">
-    <xacro:property name = "base_length" value = "0.6"/>
-    <xacro:property name = "base_width" value = "0.4"/>
-    <xacro:property name = "base_height" value = "0.2"/>
-    <xacro:property name = "wheel_radius" value = "0.1"/>
-    <xacro:property name = "wheel_length" value = "0.05"/>
-    <material name="green">
-        <color rgba="0 0.5 0 1" />
-    </material>
-    <material name="grey">
-        <color rgba="0.5 0.5 0.5 1" />
-    </material>
-    <link name="base_footprint_link">
-    </link>
-    <link name="base_link">
-        <visual>
-            <geometry>
-                <box size="${base_length} ${base_width} ${base_height}" />
-            </geometry>
-            <origin xyz="0 0 0.1" rpy="0 0 0"/>
-            <material name="green" />
-        </visual>
-    </link>
-    <xacro:macro name="wheel_link" params="prefix">
-        <link name="${prefix}_rear_wheel_link">
-            <visual>
-                <geometry>
-                    <cylinder radius = "${wheel_radius}" length = "${wheel_length}" />
-                </geometry>
-                <origin xyz="0 0 0" rpy="${pi/2.0} 0 0"/>
-                <material name="grey" />
-            </visual>
-        </link>
-    </xacro:macro>
-    <xacro:wheel_link prefix="right" />
-    <xacro:wheel_link prefix="left" />
-    <link name="front_castor_wheel_link">
-        <visual>
-            <geometry>
-                <sphere radius = "${wheel_radius/2}" />
-            </geometry>
-            <origin xyz="0 0 0" rpy="${pi/2.0} 0 0"/>
-            <material name="grey" />
-        </visual>
-    </link>
-    <joint name = "base_right_rear_wheel_joint" type="continuous">
-        <parent link = "base_link"/>
-        <child link = "right_rear_wheel_link"/>
-        <origin xyz = "${-base_length / 4.0} ${(base_width + wheel_length)/2.0} 0" rpy = "0 0 0"/>
-        <axis xyz = "0 1 0" />
-    </joint>
-    <joint name = "base_left_rear_wheel_joint" type="continuous">
-        <parent link = "base_link"/>
-        <child link = "left_rear_wheel_link"/>
-        <origin xyz = "${-base_length / 4.0} ${-(base_width + wheel_length)/2.0} 0" rpy = "0 0 0"/>
-        <axis xyz = "0 1 0" />
-    </joint>
-    <joint name = "base_front_castor_wheel_link" type="continuous">
-        <parent link = "base_link"/>
-        <child link = "front_castor_wheel_link"/>
-        <origin xyz = "${base_length / 3.0} 0 ${-wheel_radius/2}" rpy = "0 0 0"/>
-        <axis xyz = "0 1 0" />
-    </joint>
-    <joint name = "base_base_footprint_link" type="fixed">
-        <parent link = "base_footprint_link"/>
-        <child link = "base_link"/>
-        <origin xyz = "0 0 ${wheel_radius}" rpy = "0 0 0"/>
-    </joint>
+    <xacro:include filename="common_properties.xacro"/>
+    <xacro:include filename="mobile_base.xacro"/>
 </robot>
