Commit message: added intertia tags

File: src/my_robot_description/urdf/mobile_base.xacro (robot description, xacro)
@@ -16,4 +16,10 @@
             <material name="green" />
         </visual>
+        <collision>
+            <geometry>
+                <box size="${base_length} ${base_width} ${base_height}" />
+            </geometry>
+            <origin xyz="0 0 0.1" rpy="0 0 0"/>
+        </collision>
         <xacro:box_inertia m="5.0" l="${base_length}" w = "${base_height}" h ="${base_height}"
                            xyz="0 0 ${base_length}" rpy ="0 0 0" />
@@ -28,4 +34,10 @@
                 <material name="grey" />
             </visual>
+            <collision>
+                <geometry>
+                    <cylinder radius = "${wheel_radius}" length = "${wheel_length}" />
+                </geometry>
+                <origin xyz="0 0 0" rpy="${pi/2.0} 0 0"/>
+            </collision>
             <xacro:cylinder_inertia m="1.0" r="${wheel_radius}" h="${wheel_length}"
                                     xyz="0 0 0" rpy="${pi/2.0} 0 0" />
@@ -42,4 +54,10 @@
             <material name="grey" />
         </visual>
+        <collision>
+            <geometry>
+                <sphere radius = "${wheel_radius/2.0}" />
+            </geometry>
+            <origin xyz="0 0 0" rpy="${pi/2.0} 0 0"/>
+        </collision>
         <xacro:sphere_inertia m="0.5" r="${wheel_radius/2.0}"
                                 xyz="0 0 0" rpy="0 0 0" />

Commit message: some edits

File: src/my_robot_description/urdf/mobile_base.xacro (robot description, xacro)
@@ -6,6 +6,5 @@
     <xacro:property name = "wheel_radius" value = "0.1"/>
     <xacro:property name = "wheel_length" value = "0.05"/>
-    <link name="base_footprint_link">
-    </link>
+    <link name="base_footprint_link"/>
     <link name="base_link">
         <visual>
@@ -22,6 +21,6 @@
             <origin xyz="0 0 0.1" rpy="0 0 0"/>
         </collision>
-        <xacro:box_inertia m="5.0" l="${base_length}" w = "${base_height}" h ="${base_height}"
-                           xyz="0 0 ${base_length}" rpy ="0 0 0" />
+        <xacro:box_inertia m="5.0" l="${base_length}" w = "${base_height}" h ="${2*base_height}"
+                           xyz="0 0 ${base_height}" rpy ="0 0 0" />
     </link>
     <xacro:macro name="wheel_link" params="prefix">

File: src/my_robot_description/urdf/my_robot.urdf.xacro (robot description, xacro)
@@ -3,3 +3,4 @@
     <xacro:include filename="common_properties.xacro"/>
     <xacro:include filename="mobile_base.xacro"/>
+    <xacro:include filename="mobile_base_gazebo.xacro"/>
 </robot>
