Commit message: added inertial tag

File: src/my_robot_description/urdf/common_properties.xacro (robot description, xacro)
@@ -7,3 +7,12 @@
         <color rgba="0.5 0.5 0.5 1" />
     </material>
+    <xacro:macro name="box_inertia" params="m l w h xyz rpy">
+        <inertial>
+            <origin xyz="${xyz}" rpy="${rpy}" />
+            <mass value="${m}" />
+            <inertia ixx = "$(m/12)*(h*h+l*l)" ixy="0" ixz="0"
+                     iyy = "$(m/12)*(w*w+l*l)" iyz = "0"
+                     izz = "$(m/12)*(w*w+h*h)" />
+        </inertial>
+    </xacro:macro>
 </robot>

File: src/my_robot_description/urdf/mobile_base.xacro (robot description, xacro)
@@ -16,4 +16,6 @@
             <material name="green" />
         </visual>
+        <xacro:box_inertia m="5.0" l="${base_length}" w = "${base_hheight}" h ="${base_height}"
+                           xyz="0 0 ${base_length}" rpy ="0 0 0" />
     </link>
     <xacro:macro name="wheel_link" params="prefix">

Commit message: added intertia tags

File: src/my_robot_description/urdf/common_properties.xacro (robot description, xacro)
@@ -11,7 +11,25 @@
             <origin xyz="${xyz}" rpy="${rpy}" />
             <mass value="${m}" />
-            <inertia ixx = "$(m/12)*(h*h+l*l)" ixy="0" ixz="0"
-                     iyy = "$(m/12)*(w*w+l*l)" iyz = "0"
-                     izz = "$(m/12)*(w*w+h*h)" />
+            <inertia ixx = "${(m/12)*(h*h+l*l)}" ixy="0" ixz="0"
+                     iyy = "${(m/12)*(w*w+l*l)}" iyz = "0"
+                     izz = "${(m/12)*(w*w+h*h)}" />
+        </inertial>
+    </xacro:macro>
+    <xacro:macro name="cylinder_inertia" params="m r h xyz rpy">
+        <inertial>
+            <origin xyz="${xyz}" rpy="${rpy}" />
+            <mass value="${m}" />
+            <inertia ixx = "${(m/12)*3*(r*r+h*h)}" ixy="0" ixz="0"
+                     iyy = "${(m/12)*3*(r*r+h*h)}" iyz = "0"
+                     izz = "${(m/2)*(r*r)}" />
+        </inertial>
+    </xacro:macro>
+    <xacro:macro name="sphere_inertia" params="m r xyz rpy">
+        <inertial>
+            <origin xyz="${xyz}" rpy="${rpy}" />
+            <mass value="${m}" />
+            <inertia ixx = "${(2/5)*m*r*r}" ixy="0" ixz="0"
+                     iyy = "${(2/5)*m*r*r}" iyz = "0"
+                     izz = "${(2/5)*m*r*r}" />
         </inertial>
     </xacro:macro>

File: src/my_robot_description/urdf/mobile_base.xacro (robot description, xacro)
@@ -16,5 +16,5 @@
             <material name="green" />
         </visual>
-        <xacro:box_inertia m="5.0" l="${base_length}" w = "${base_hheight}" h ="${base_height}"
+        <xacro:box_inertia m="5.0" l="${base_length}" w = "${base_height}" h ="${base_height}"
                            xyz="0 0 ${base_length}" rpy ="0 0 0" />
     </link>
@@ -28,4 +28,6 @@
                 <material name="grey" />
             </visual>
+            <xacro:cylinder_inertia m="1.0" r="${wheel_radius}" h="${wheel_length}"
+                                    xyz="0 0 0" rpy="${pi/2.0} 0 0" />
         </link>
     </xacro:macro>
@@ -35,9 +37,11 @@
         <visual>
             <geometry>
-                <sphere radius = "${wheel_radius/2}" />
+                <sphere radius = "${wheel_radius/2.0}" />
             </geometry>
             <origin xyz="0 0 0" rpy="${pi/2.0} 0 0"/>
             <material name="grey" />
         </visual>
+        <xacro:sphere_inertia m="0.5" r="${wheel_radius/2.0}"
+                                xyz="0 0 0" rpy="0 0 0" />
     </link>
     <joint name = "base_right_rear_wheel_joint" type="continuous">

Commit message: restarting on project

File: src/my_robot_description/urdf/common_properties.xacro (robot description, xacro)
@@ -11,7 +11,7 @@
             <origin xyz="${xyz}" rpy="${rpy}" />
             <mass value="${m}" />
-            <inertia ixx = "${(m/12)*(h*h+l*l)}" ixy="0" ixz="0"
-                     iyy = "${(m/12)*(w*w+l*l)}" iyz = "0"
-                     izz = "${(m/12)*(w*w+h*h)}" />
+            <inertia ixx = "${(m/12)*(w*w+h*h)}" ixy="0" ixz="0"
+                     iyy = "${(m/12)*(l*l+w*w)}" iyz = "0"
+                     izz = "${(m/12)*(h*h+l*l)}" />
         </inertial>
     </xacro:macro>

File: src/my_robot_description/urdf/mobile_base.xacro (robot description, xacro)
@@ -19,8 +19,8 @@
                 <box size="${base_length} ${base_width} ${base_height}" />
             </geometry>
-            <origin xyz="0 0 0.1" rpy="0 0 0"/>
+            <origin xyz="0 0 ${base_height/2.0}" rpy="0 0 0"/>
         </collision>
         <xacro:box_inertia m="5.0" l="${base_length}" w = "${base_height}" h ="${2*base_height}"
-                           xyz="0 0 ${base_height}" rpy ="0 0 0" />
+                           xyz="0 0 ${base_height/2.0}" rpy ="0 0 0" />
     </link>
     <xacro:macro name="wheel_link" params="prefix">
@@ -35,7 +35,7 @@
             <collision>
                 <geometry>
-                    <cylinder radius = "${wheel_radius}" length = "${wheel_length}" />
+                    <sphere radius="${wheel_radius}" />
                 </geometry>
-                <origin xyz="0 0 0" rpy="${pi/2.0} 0 0"/>
+                <origin xyz="0 0 0" rpy="0 0 0"/>
             </collision>
             <xacro:cylinder_inertia m="1.0" r="${wheel_radius}" h="${wheel_length}"
